File: PiPower_v2_bak.kicad_pcb (KiCad board)
At the start: 2 copper layers, 56 x 60 mm, 80 parts, among them J1 MicroUSB_in, J10 5V_Pi, J11 12V_Out, J12 5V_IN, J2 LiPo_JST, J3 USB_A_out, J4 Auto_On, J5 5V_USB, J6 5V_EXT, J7 5V_OUT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

Commit message: 1311031620 Schematic complete, needs to be verified
Parts:
- removed D8: 5V_Pi, led_0805
- removed J12: 5V_IN, Header_3
- removed L2: 2u2H,1.9A, Inductor_SMD2
- removed R23: 470k, r_0805
- removed R6: 4k7, r_0805
- removed SJ2: 5V_OUT, ShortLink
- removed SJ5: STAT, ShortLink2
- added D1: LSM115J, diode-DO214BA, F.Cu at (112.2, 20.8)
- added D5: LSM115J, diode-DO214BA, F.Cu at (133.1, 72.7)
- added Q1: 2SK3019, SOT416_2SK3019, F.Cu at (134.7, 66.5)
- added R7: 10k, r_0805, F.Cu at (135.6, 62.1)
- C10, C18, C9: footprint c_1206 -> c_0805
- C14: value 10uF X7R -> 10uF; footprint c_1206 -> C_ELCO_SMD
- C2: value 10uF X7R -> 100u,25V; footprint c_1206 -> C_ELCO_SMD
- C3: value 22uF X7R -> 2u2 Tant; footprint c_1210 -> c_0805
- C5, C6: value 10uF X7R -> 10u; footprint c_1206 -> C_ELCO_SMD
- D7: value 5V_OUT -> EXT_ON
- J7: value 5V_OUT -> 5V_IN
- R1, R2, R9: value 4k7 -> 1k5
- R3: value 4k7 -> 2k
- SJ1: value BAT -> LINK1
- U2: value TPS62163 -> NCP1117ST50; footprint TPS62163_DSG -> SOT223
Connections:
- C11 pad 2: /5V_IN -> /5V_EXT
- C12 pad 2: /5V_BAT -> /5V_USB
- C2 pad 1: /PWR_IN -> N-000001
- D3 pad 1: N-0000015 -> /STAT
- D4 pad 2: N-0000014 -> /STAT
- D6 pad 2: N-000009 (its old number) -> GND
- D7 pad 1: N-0000011 (its old number) -> /5V_IN
- H1 pad 1: N-0000045 -> (no net)
- H2 pad 1: N-0000048 -> (no net)
- J1 pad 2: N-0000039 -> (no net)
- J1 pad 3: N-0000040 -> (no net)
- J1 pad 4: N-0000041 -> (no net)
- J3 pad 2: N-0000028 -> (no net)
- J3 pad 3: N-0000029 -> (no net)
- J4 pad 3: /5V_OUT -> /5V_IN
- J7 pad 1: /5V_OUT -> /5V_IN
- P1 pad 10: N-0000046 -> (no net)
- P1 pad 11: N-0000060 -> (no net)
- P1 pad 12: N-0000052 -> (no net)
- P1 pad 13: N-0000055 -> (no net)
- P1 pad 14: N-0000070 -> (no net)
- P1 pad 15: N-0000062 -> (no net)
- P1 pad 16: N-0000061 -> (no net)
- P1 pad 17: N-0000057 -> (no net)
- P1 pad 18: N-0000058 -> (no net)
- P1 pad 19: N-0000059 -> (no net)
- P1 pad 20: N-0000069 -> (no net)
- P1 pad 21: N-0000063 -> (no net)
- P1 pad 22: N-0000066 -> (no net)
- P1 pad 23: N-0000064 -> (no net)
- P1 pad 24: N-0000065 -> (no net)
- P1 pad 25: N-0000071 -> (no net)
- P1 pad 26: N-0000056 -> (no net)
- P1 pad 4: N-0000067 -> (no net)
- P1 pad 8: N-0000047 -> (no net)
- P1 pad 9: N-0000068 -> (no net)
- Q2 pad 3: /5V_OUT -> /5V_IN
- R18 pad 1: /5V_OUT -> /5V_IN
- R19 pad 1: /5V_OUT -> /5V_IN
- R5 pad 1: N-000008 (its old number) -> /5V_IN
- R5 pad 2: /5V_EXT -> N-000006
- SJ1 pad 1: N-000009 (its old number) -> /5V_IN
- SJ1 pad 2: GND -> /5V_BAT
- U2 pad 2: /PWR_IN -> /5V_EXT
- U2 pad 3: /PWR_IN -> N-000001
- U3 pad 6: /5V_BAT -> /5V_USB
- U3 pad 7: /5V_OUT -> /5V_IN
- U3 pad 8: /5V_IN -> /5V_EXT
- U4 pad 6: /VBAT -> /EN
Routing:
- net /5V_IN: track 37.3 -> 116.2 mm, vias 2 -> 4
- net GND: track 410.0 -> 445.5 mm
- net /5V_EXT: track 3.18 -> 37.4 mm
- net /5V_BAT: track 14.9 -> 40.6 mm
- net /5V_USB: track 16.1 -> 40.2 mm, vias 0 -> 1
- net /5V_OUT: track 23.6 -> 0.00 mm, vias 1 -> 0
- net N-000001: track 0.00 -> 17.1 mm
- net /EN: track 0.00 -> 11.6 mm
- net /VBAT: track 74.1 -> 84.7 mm
- net /PWR_IN: track 66.6 -> 71.4 mm
- net /STAT: track 0.00 -> 4.12 mm
- net N-0000014: track 1.95 -> 0.00 mm
- net N-000006: track 0.00 -> 1.93 mm
- added copper zone on F.Cu, net /5V_BAT
- added copper zone on F.Cu, net /5V_EXT
- added copper zone on F.Cu, net /VBAT
- added copper zone on F.Cu, net GND
