File: PiPower_v2.sch (KiCad schematic (older format))
At the start: 81 parts, among them J1 MicroUSB_in, J10 5V_Pi, J11 12V_Out, J12 5V_IN, J2 LiPo_JST, J3 USB_A_out, J4 Auto_On, J5 5V_USB, J6 5V_EXT, J7 5V_OUT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

Commit message: new BoM work in progress
Parts:
- C10, C14, C18, C2, C5, C6, C9: footprint C_ELCO_SMD -> c_1206
- C3: footprint c_0805 -> c_1210
- J12: footprint (none) -> Header_3
- L2: footprint Inductor_SMD1 -> Inductor_SMD2
- P1: footprint Header_GPIO -> Header_GPIO_3
- SJ5: footprint (none) -> ShortLink2
- U2: footprint (none) -> TPS62163_DSG
Changed lines of the file:
@@
 Sheet 1 1
 Title "uControl_POWER"
-Date "1 oct 2013"
+Date "20 nov 2013"
 Rev "v1"
 Comp "WyoLum"
@@
 F 0 "C14" H 9225 3475 40  0000 C CNN
 F 1 "10uF X7R" H 9250 3300 40  0000 C CNN
-F 2 "C_ELCO_SMD" H 9075 3400 60  0001 C CNN
+F 2 "c_1206" H 9075 3400 60  0001 C CNN
 F 3 "" H 9075 3400 60  0000 C CNN
 	1    9075 3400
@@
 F 0 "C5" H 1825 4625 40  0000 C CNN
 F 1 "10uF X7R" V 1700 4800 40  0000 C CNN
-F 2 "C_ELCO_SMD" H 1775 4525 60  0001 C CNN
+F 2 "c_1206" H 1775 4525 60  0001 C CNN
 F 3 "" H 1775 4525 60  0000 C CNN
 	1    1775 4525
@@
 F 0 "C6" H 4200 4600 40  0000 C CNN
 F 1 "10uF X7R" V 4250 4350 39  0000 C CNN
-F 2 "C_ELCO_SMD" H 4150 4525 60  0001 C CNN
+F 2 "c_1206" H 4150 4525 60  0001 C CNN
 F 3 "" H 4150 4525 60  0000 C CNN
 	1    4150 4525
@@
 F 0 "C9" H 1425 6800 40  0000 C CNN
 F 1 "10uF X7R" V 1425 6550 40  0000 C CNN
-F 2 "C_ELCO_SMD" H 1375 6725 60  0001 C CNN
+F 2 "c_1206" H 1375 6725 60  0001 C CNN
 F 3 "" H 1375 6725 60  0000 C CNN
 	1    1375 6725
@@
 F 0 "C10" H 4500 6800 40  0000 C CNN
 F 1 "10uF X7R" V 4500 6550 40  0000 C CNN
-F 2 "C_ELCO_SMD" H 4450 6725 60  0001 C CNN
+F 2 "c_1206" H 4450 6725 60  0001 C CNN
 F 3 "" H 4450 6725 60  0000 C CNN
 	1    4450 6725
@@
 F 0 "C2" H 2050 2625 40  0000 C CNN
 F 1 "10uF X7R" V 2050 2300 40  0000 C CNN
-F 2 "C_ELCO_SMD" H 2000 2550 60  0001 C CNN
+F 2 "c_1206" H 2000 2550 60  0001 C CNN
 F 3 "" H 2000 2550 60  0000 C CNN
 	1    2000 2550
@@
 F 0 "C3" H 3975 2650 40  0000 C CNN
 F 1 "22uF X7R" V 3950 2300 40  0000 C CNN
-F 2 "c_0805" H 3900 2550 60  0001 C CNN
+F 2 "c_1210" H 3900 2550 60  0001 C CNN
 F 3 "" H 3900 2550 60  0000 C CNN
 	1    3900 2550
@@
 F 0 "P1" H 10425 6850 40  0000 C CNN
 F 1 "RASPI_GPIO" V 10325 6150 40  0000 C CNN
-F 2 "Header_GPIO" H 10425 6150 60  0001 C CNN
+F 2 "Header_GPIO_3" H 10425 6150 60  0001 C CNN
 F 3 "" H 10425 6150 60  0000 C CNN
 	1    10325 6150
@@
 F 0 "C18" H 4350 6800 40  0000 C CNN
 F 1 "10uF X7R" V 4350 6550 40  0000 C CNN
-F 2 "C_ELCO_SMD" H 4300 6725 60  0001 C CNN
+F 2 "c_1206" H 4300 6725 60  0001 C CNN
 F 3 "" H 4300 6725 60  0000 C CNN
 	1    4300 6725
@@
 F 0 "U2" H 2575 3175 40  0000 L BNN
 F 1 "TPS62163" H 2375 2400 40  0000 L TNN
-F 2 "" H 2625 3050 60  0000 C CNN
+F 2 "TPS62163_DSG" H 2625 3050 60  0001 C CNN
 F 3 "" H 2625 3050 60  0000 C CNN
 	1    2625 2750
@@
 F 0 "L2" V 3325 2400 40  0000 C CNN
 F 1 "2u2H,1.9A" V 3475 2400 40  0000 C CNN
-F 2 "Inductor_SMD1" H 3375 2400 60  0001 C CNN
+F 2 "Inductor_SMD2" H 3375 2400 60  0001 C CNN
 F 3 "~" H 3375 2400 60  0000 C CNN
 F 4 "VLF3012ST-2R2M1R4" V 3550 2425 40  0000 C CNN "Mfr_PN"
@@
 F 0 "SJ5" H 2675 4200 40  0000 C CNN
 F 1 "STAT" H 2775 4375 40  0000 C CNN
-F 2 "" H 2750 4300 60  0000 C CNN
+F 2 "ShortLink2" H 2750 4300 60  0001 C CNN
 F 3 "" H 2750 4300 60  0000 C CNN
 	1    2775 4300
@@
 F 0 "J12" V 4675 1400 40  0000 C CNN
 F 1 "5V_IN" V 4775 1400 40  0000 C CNN
-F 2 "" H 4725 1400 60  0000 C CNN
+F 2 "Header_3" H 4725 1400 60  0001 C CNN
 F 3 "" H 4725 1400 60  0000 C CNN
 	1    4725 1400
